Commit message: Move Robot to location is localized and working

File: src/my_robot_description/urdf/mobile_base.xacro (robot description, xacro)
@@ -35,7 +35,7 @@
                 <collision>
                     <geometry>
-                        <sphere radius="${wheel_radius}" />
+                        <cylinder radius="${wheel_radius}" length="${wheel_length}" />
                     </geometry>
-                    <origin xyz="0 0 0" rpy="0 0 0" />
+                    <origin xyz="0 0 0" rpy="${pi / 2.0} 0 0" />
                 </collision>
                 <xacro:cylinder_inertia m="1.0" r="${wheel_radius}" l="${wheel_length}" o_xyz="0 0 0" o_rpy="${pi / 2.0} 0 0" />

File: src/my_robot_description/urdf/mobile_base_gazebo.xacro (robot description, xacro)
@@ -22,14 +22,21 @@
                 <wheel_separation>0.45</wheel_separation>
                 <wheel_radius>0.1</wheel_radius>
-                <max_wheel_torque>20</max_wheel_torque>
-                <max_wheel_acceleration>1.0</max_wheel_acceleration>
-                <odom_frame>${robot_name}_odom</odom_frame>
-                <robot_base_frame>${robot_name}_base_footprint</robot_base_frame>
+                <max_wheel_torque>200</max_wheel_torque>
+                <max_wheel_acceleration>10.0</max_wheel_acceleration>
                 <topic>/model/${robot_name}/cmd_vel</topic>
-                <odom_topic>/model/${robot_name}/odometry</odom_topic>
-                <tf_topic>/model/${robot_name}/tf</tf_topic>
-                <publish_odom>true</publish_odom>
-                <publish_odom_tf>true</publish_odom_tf>
-                <publish_wheel_tf>true</publish_wheel_tf>
+            </plugin>
+        </gazebo>
+        <!-- Pose Publisher Plugin (simulates GPS with exact positioning) -->
+        <gazebo>
+            <plugin
+                filename="gz-sim-pose-publisher-system"
+                name="gz::sim::systems::PosePublisher">
+                <publish_link_pose>true</publish_link_pose>
+                <publish_collision_pose>false</publish_collision_pose>
+                <publish_visual_pose>false</publish_visual_pose>
+                <use_pose_vector_msg>true</use_pose_vector_msg>
+                <static_publisher>true</static_publisher>
+                <static_update_frequency>10</static_update_frequency>
+                <link_name>${robot_name}_base_footprint</link_name>
             </plugin>
         </gazebo>
@@ -38,5 +45,5 @@
                 filename="gz-sim-joint-state-publisher-system"
                 name="gz::sim::systems::JointStatePublisher">
-                <topic>/world/empty/model/${robot_name}/joint_state</topic>
+                <topic>${robot_name}/joint_state</topic>
             </plugin>
         </gazebo>

File: src/my_robot_description/urdf/my_robot.urdf.xacro (robot description, xacro)
@@ -22,5 +22,5 @@
         <parent link="world_base_footprint" />
         <child link="${robot_name}_base_footprint" />
-        <origin xyz="${robot_x} ${robot_y} ${robot_z}" rpy="0 0 ${robot_yaw}" />
+        <origin xyz="0 0 0" rpy="0 0 ${robot_yaw}" />
     </joint>
     <!-- Instantiate the mobile base with robot name -->
